File: internal/boardfamily/reference-sht31/board.kicad_pcb (KiCad board)
At the start: 2 copper layers, 120 x 80 mm, 16 parts, among them J1 Conn_01x02, J2 UART PROG, J3 GPIO I2C SPI, SW1 RESET, SW2 BOOT, U1 ESP32-WROOM-32E, U2 SHT31-DIS-B 0x44

Commit message: Qualify SHT31 assembly reference and publish two-family examples
Parts:
- U2: footprint Sensor_Humidity:Sensirion_DFN-8-1EP_2.5x2.5mm_P0.5mm_EP1.1x1.7mm -> Sensor_Humidity:SHT31-DIS_SensirionV7_MaskPaste
